Commit message: adt_hardware

File: src/adt_hardware/description/ros2_control/diffbot.ros2_control.xacro (robot description, xacro)
@@ -1,9 +1,9 @@
 <?xml version="1.0"?>
 <robot xmlns:xacro="http://www.ros.org/wiki/xacro">
-  <xacro:macro name="diffbot_ros2_control" params="name prefix use_mock_hardware">
+  <xacro:macro name="service_roboter_ros2_control" params="name prefix use_mock_hardware">
     <ros2_control name="${name}" type="system">
       <xacro:unless value="${use_mock_hardware}">
         <hardware>
-          <plugin>ADT_HARDWARE/ArduinoSerialBridge</plugin>
+          <plugin>adt_hardware/BasisMotorSerialBridge</plugin>
           <param name="example_param_hw_start_duration_sec">0</param>
           <param name="example_param_hw_stop_duration_sec">3.0</param>

File: src/adt_hardware/description/urdf/diffbot.urdf.xacro (robot description, xacro)
@@ -4,11 +4,10 @@
   <xacro:arg name="prefix" default="" />
   <xacro:arg name="use_mock_hardware" default="false" />
-  <xacro:include filename="$(find ros2_control_demo_description)/diffbot/urdf/diffbot_description.urdf.xacro" />
+  <xacro:include filename="$(find ros2_control_demo_description)/service_roboter/urdf/service_roboter_description.urdf.xacro" />
   <!-- Import Rviz colors -->
-  <xacro:include filename="$(find ros2_control_demo_description)/diffbot/urdf/diffbot.materials.xacro" />
-  <!-- Import diffbot ros2_control description -->
-  <xacro:include filename="$(find ADT_HARDWARE)/ros2_control/diffbot.ros2_control.xacro" />
-  <xacro:diffbot prefix="$(arg prefix)" />
-  <xacro:diffbot_ros2_control
-    name="DiffBot" prefix="$(arg prefix)" use_mock_hardware="$(arg use_mock_hardware)"/>
+  <xacro:include filename="$(find ros2_control_demo_description)/service_roboter/urdf/service_roboter.materials.xacro" />
+  <!-- Import service_roboter ros2_control description -->
+  <xacro:include filename="$(find adt_hardware)/ros2_control/service_roboter.ros2_control.xacro" />
+  <xacro:service_roboter prefix="$(arg prefix)" />
+  <xacro:service_roboter_ros2_control name="service_roboter" prefix="$(arg prefix)" use_mock_hardware="$(arg use_mock_hardware)"/>
 </robot>
